File: Hardware/PCB/serial_spi_lcd.kicad_sch (KiCad schematic)
At the start: 3 parts, among them U1 ER-TFTM032-3

Commit message: kinda pricey, I should try to make a smaller version using LCSC parts for cheaper solution
Parts:
- C16: LCSC (none) -> C307520
- C23: LCSC (none) -> C66501
Changed lines of the file:
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@@
 			"fwAAiJ1Kn/t/AACgWjoBcgIAAHAeOgFyAgAAML5Kn/t/AACQHjoBcgIAANBaOgFyAgAAiJ1Kn/t/"
 			"AACQu0qf+38AAIidSp/7fwAAAFs6AXICAACwHjoBcgIAADC+Sp/7fwAA0B46AXICAAAwWzoBcgIA"
-			"AIidSp/7fwAAkLtKn/t/AACInUqf+38AAGBbOgFyAgAA8B46AXICAAAwvkqf+38AAA=="
+			"AIidSp/7fwAAkLtKn/t/AACInUqf+38AAGBbOgFyAgAA8B46AXICAAAwvkqf+38AAFUATgBLAG8A"
+			"VQBxAFUAUwBNAGkASQAvAEkAdgBxAGIAUQB6AHMAZgAwAFMAKwBmADQAVgAxAGkAQwBZAC8ANQAv"
+			"AEMAaABjAFgAZABJAGQAbgBSAFoAKwBoAEsAWABUAFIAVwB6AHUAbgB2AFAAYgBVAHgAdwBKAEsA"
+			"SABaAFkAagBQAE8AaQBkAFQAOQBCADgAagA0ADYAVwBYAGgAUgBUAGwASgAvAEEARgBiAHYAWAB3"
+			"AHUAYgB1AHMASQBhAHMANgBEAEsAYgBJAEcAcABnAHcAdwBSAGUAdgBPAEcANABLAFMASABqAHkA"
+			"aQAzADQANwBnAFkARwA0ADEAVABOAG4AcABRAFUAMQBPAEQAbQB2ADQARQBlAEMAYgBFADQALwBL"
+			"AGgAawA4AEkAQgBQAGkAWABrADUAUwBBAHIAVwBRADMAOQBwAGcAeQBCAHMAUABHAEgAVgBGAFgA"
+			"MABHAE4AOABQAFYAWgAvAGYAeABOADAAdgBGAGEAQQBzACsATQAxAE0AVABVADMASgB1ADgAcgBM"
+			"AFQAMABWAEsATwBnAGUASwBpAGcAbwBsADMANwA4AC8AdgBPADIAVQBuAEUANQBMAEQASABjADQA"
+			"aABRADAAOQBOAFMASABCAFQANABHAFUAbABpAEYAMABzAHQAOQBxAEEAVQBtAG8AMQBhAG8ARwBW"
+			"AFYAVgBUAHIAUABZADQAaABmAGsAOQBqAEsARABKAE4AQQB1AFMAVgBFAFAAVABvAGMAcwB3AHQA"
+			"NQBkAHUAWABtAEMASgArAHUAVQA0AGwAUgByAEQAdABGAEUAbAA5AGgANQBMAHoAaABCAEwAegBy"
+			"ADUARwBKAHAAKwBQADEAQgBjAG4AWQBEAHYAYQBGAEQAVQBLAG4AcAB3AHEAMQBFAEgAWABzAFUA"
+			"dQBFAFoAWgBJAEQAbgBiAEYAMABnAGoAbABFAEcAbQBhAFUAUwBiAC8AMwArADEAegBSAEEAagBZ"
+			"ADkAdQBmAEIAeQA5AHMASABEAFUAMgBmAHgAMABYAHcANAArAG4AOQA3ADUAdgAyAE4AUgBCADgA"
+			"MwArAEgAeABwAEEASABOAFQATABUAFoASABqAEUAUQBmAHUAUABsADgAUQBRAE4AegBVADIAaABK"
+			"ADYANgBKAFYAdgA4AEUAWQBNAG0AUgBJAGcAVABRAEEANwBhAG8ASgBqAHIAYQBKAGQANwBCAHIA"
+			"MwBpAHEANABpAHcANgBOAG4ASgBHAEYATABBAGsANQB5AE0AdQB6AFgANwBVAGYAWABOAGMAaQBa"
+			"AGQANwBHAFUAagBNAHoATABNADcAcAAyADUAdgBGAHYASwBhAHMANABEAFcAegA3AAAAAAAAAAAA"
+			"AAAAAAAAAAAAAAAAAAAAAAAAAAAAAAAAAAAAAAAAAAAAAAAAAAAAAAAAAAAAAAAAAAAAAAAAAAAA"
+			"AAAAAAAAAAAAAAAAAAAAAAAAAAAAAAAAAAAAAAAAAAAAAAAAAAAAAAAAAAAAAAAAAAAAAAAAAAAA"
+			"AAAAAAAAAAAAAAAAAAAAAAAAAAAAAAAAAAAAAAAAAAAAAAAAAAAAAAAAAAAAAAAAAAAAAAAAAAAA"
+			"AAAAAAAAAAAAAAAAAAAAAAAAAAAAAAAAAAAAAAAAAAAAAAAAAAAAAAAAAAAAAAAAAAAAAAAAAAAA"
+			"AAAAAAAAAAAAAAAAAAAAAAAAAAAAAAAAAAAAAAAAAAAAAAAAAAAAAAAAAAAAAAAAAAAAAAAAAAAA"
+			"AAAAAAAAAAAAAAAAAAAAAAAAAAAAAAAAAAAAAAAAAAAAAAAAAAAAAAAAAAAAAAAAAAAAAAAAAAAA"
+			"AAAAAAAAAAAAAAAAAAAAAAAAAAAAAAAAAAAAAAAAAAAAAAAAAAAAAAAAAAAAAAAAAAAAAAAAAAAA"
+			"AAAAAAAAAAAAAAAAAAAAAAAAAAAAAAAAAAAAAAAAAAAAAAAAAAAAAAAAAAAAAAAAAAAAAAAAAAAA"
+			"AAAAAAAAAAAAAAAAAAAAAAAAAAAAAAAAAAAAAAAAAAAAAAAAAAAAAAAAAAAAAAAAAAAAAAAAAAAA"
+			"AAAAAAAAAAAAAAAAAAAAAAAAAAAAAAAAAAAAAAAAAAAAAAAAAAAAAAAAAAAAAAAAAAAAAAAAAAAA"
+			"AAAAAAAAAAAAAAAAAAAAAAAAAAAAAAAAAAAAAAAAAAAAAAAAAAAAAAAAAAAAAAAAAAAAAAAAAAAA"
+			"AAAAAAAAAAAAAAAAAAAAAAAAAAAAAAAAAAAAAAAAAAAAAAAAAAAAAAAAAAAAAAAAAAAAAAAAAAAA"
+			"AAAAAAAAAAAAAAAAAAAAAAAAAAAAAAAAAAAAAAAAAAAAAAAAAAAAAAAAAAAAAAAAAAAAAAAAAAAA"
+			"AAAAAAAAAAAAAAAAAAAAAAAAAAAAAAAAAAAAAAAAAAAAAAAAAAAAAAAAAAAAAAAAAAAAAAAAAAAA"
+			"AAAAAAAAAAAAAAAAAAAAAAAAAAAAAAAAAAAAAAAAAAAAAAAAAAAAAAAAAAAAAAAAAAAAAAAAAAAA"
+			"AAAAAAAAAAAAAAAAAAAAAAAAAAAAAAAAAAAAAAAAAAAAAAAAAAAAAAAAAAAAAAAAAAAAAAAAAAAA"
+			"AAAAAAAAAAAAAAAAAAAAAAAAAAAAAAAAAAAAAAAAAAAAAAAAAAAAAAAAAAAAAAAAAAAAAAAAAAAA"
+			"AAAAAAAAAAAAAAAAAAAAAAAAAAAAAAAAAAAAAAAAAAAAAAAAAAAAAAAAAAAAAAAAAA=="
 		)
 	)
@@
 			)
 		)
+		(property "LCSC" "C66501"
+			(at 80.01 54.61 0)
+			(effects
+				(font
+					(size 1.27 1.27)
+				)
+			)
+		)
 		(pin "1"
 		)
@@
 			)
 		)
+		(property "LCSC" "C307520"
+			(at 71.12 54.61 0)
+			(effects
+				(font
+					(size 1.27 1.27)
+				)
+			)
+		)
 		(pin "2"
 		)
@@
 			)
 		)
+		(property "LCSC" ""
+			(at 104.14 49.53 0)
+			(effects
+				(font
+					(size 1.27 1.27)
+				)
+			)
+		)
